File: ESP32_Sheald.kicad_pcb (KiCad board)
At the start: 4 copper layers, 69 x 40.6 mm, 34 parts, among them J1 BME280, SHT40 Module, J10 SCD40 Module, J11 Conn_01x03, J2 SCD40 Module, J3 Conn_01x02, J4 Qwiic_Vertical, J5 Conn_01x02, J6 Conn_01x02, J7 Conn_01x03, J8 Conn_01x03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

Commit message: working kibotfile for gerber
Routing:
- net SCK: track 55.6 -> 122.2 mm, vias 1 -> 3
- net PhotoMeas: track 3.80 -> 64.6 mm, vias 0 -> 1
- net SDA: track 67.9 -> 124.4 mm, vias 1 -> 2
- net Net-(U1-GP1): track 0.00 -> 55.7 mm
- net Net-(U1-GP2): track 0.00 -> 45.3 mm
- net +5V: track 44.8 -> 76.5 mm
