File: ESP32_Sheald.kicad_pcb (KiCad board)
At the start: 4 copper layers, 69 x 40.6 mm, 34 parts, among them J1 BME280, SHT40 Module, J10 SCD40 Module, J11 Conn_01x03, J2 SCD40 Module, J3 Conn_01x02, J4 Qwiic_Vertical, J5 Conn_01x02, J6 Conn_01x02, J7 Conn_01x03, J8 Conn_01x03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

Commit message: ready for order
Parts:
- removed JP1: SolderJumper_2_Open, Jumper:SolderJumper-2_P1.3mm_Open_TrianglePad1.0x1.5mm
- added J12: Conn_01x03, PCM_SparkFun-Connector:1x03_P2.54mm, F.Cu at (107.5, 102.8)
- added R11: 470R, Resistor_SMD:R_0805_2012Metric, F.Cu at (110.2, 102.0)
- added R12: 470R, Resistor_SMD:R_0805_2012Metric, F.Cu at (117.8, 100.8)
- C1, C6: footprint Capacitor_SMD:C_0603_1608Metric -> Capacitor_SMD:C_0805_2012Metric
- R1, R2: value R -> 4k7
- moved R10 1.25 mm to (112.8, 102.0)
- moved R1 1.12 mm to (152.0, 102.5), turned to 90 degrees
- moved R2 0.41 mm to (144.8, 102.0), turned to 90 degrees
- moved C6 0.35 mm to (155.2, 91.8)
Connections:
- net Net-(JP1-B) renamed GPIO_5
- net Net-(U1-GP1) renamed GPIO_1
- net Net-(U1-GP13) renamed PIR
- net Net-(U1-GP2) renamed GPIO_2
- R1 pad 1: +3V3 -> Net-(J6-Pin_2)
- R1 pad 2: Net-(J6-Pin_2) -> +3V3
- R2 pad 1: +3V3 -> Net-(J5-Pin_2)
- R2 pad 2: Net-(J5-Pin_2) -> +3V3
- U1 pad 7: Net-(J7-Pin_2) -> GPIO_4
- U1 pad 9: unconnected-(U1-GP6-Pad9) -> GPIO_6
Routing:
- net Net-(J12-Pin_2): track 0.00 -> 15.1 mm, vias 0 -> 2
- net GPIO_6: track 0.00 -> 5.74 mm
- net GPIO_4: track 0.00 -> 5.61 mm
- net Net-(J7-Pin_2): track 11.4 -> 6.53 mm
- net Net-(J8-Pin_2): track 6.85 -> 3.26 mm
- net UART_TX_mmWAVE: track 11.7 -> 14.8 mm
- net GPIO_5: track 8.15 -> 5.59 mm
- net Net-(J3-Pin_2): track 19.7 -> 20.4 mm
- net GPIO_2: track 45.3 -> 44.6 mm
- net SDA: track 124.4 -> 125.1 mm
- net Net-(J3-Pin_1): track 18.6 -> 19.3 mm
- net GND: vias 1 -> 13
