File: ESP32_Sheald.kicad_sch (KiCad schematic)
At the start: 34 parts, among them J1 BME280, SHT40 Module, J10 SCD40 Module, J11 Conn_01x03, J2 SCD40 Module, J3 Conn_01x02, J4 Qwiic_Vertical, J5 Conn_01x02, J6 Conn_01x02, J7 Conn_01x03, J8 Conn_01x03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

Commit message: ready for order
Parts:
- removed JP1: SolderJumper_2_Open, Jumper:SolderJumper-2_P1.3mm_Open_TrianglePad1.0x1.5mm, symbol Jumper:SolderJumper_2_Open
- added J12: Conn_01x03, PCM_SparkFun-Connector:1x03_P2.54mm, symbol PCM_SparkFun-Connector:Conn_01x03_P2.54mm
- added R11, R12: 470R, Resistor_SMD:R_0805_2012Metric, symbol Device:R
- C1, C6: footprint Capacitor_SMD:C_0603_1608Metric -> Capacitor_SMD:C_0805_2012Metric
- R1, R2: value R -> 4k7
Connections:
- net +3V3: now also R1.2, R2.2, J12.3 (Pin_3); no longer R1.1, R2.1
- net GND: now also J12.1 (Pin_1)
- net at J5.2 (Pin_2), R8.1: now also R2.1; no longer R2.2
- net GPIO_2: now reaches R8.2, U1.5 (GP2)
- net PIR: now reaches U1.16 (GP13), U4.3 (SIGN)
- net GPIO_1: now reaches R7.2, U1.4 (GP1)
- net at J7.2 (Pin_2): now also R11.1; no longer U1.7 (GP4)
- net GPIO_5: now reaches R10.2, U1.8 (GP5)
- net GPIO_6: now reaches U1.9 (GP6)
- net GPIO_6: now also R12.2
- net at J6.2 (Pin_2), R7.1: now also R1.1; no longer R1.2
- new net: J12.2 (Pin_2), R12.1
- new net GPIO_4: R11.2, U1.7 (GP4)
Other:
- note added: "ESP32 zero module (C3, S3 , C6)"
- note added: "GPIOs"
- note added: "I2C Modules"
- note added: "PIR sensor"
- note added: "Phototransistor"
- note added: "QWIIC connector"
- note added: "SHT40 temperature and humidity"
- note added: "addressable LED"
- note added: "mmWave"
- note added: "solid state relais"
- note added: "supply pins"
- moved on the sheet: C1, C2, C3, C6, J1, J10, J11, J2, J4, J5, J6, J7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
