File: ESP32_Shield.kicad_pcb (KiCad board)
At the start: 4 copper layers, 69 x 40.6 mm, 36 parts, among them J1 BME280, SHT40 Module, J10 SCD40 Module, J11 Conn_01x03, J12 Conn_01x03, J2 SCD40 Module, J3 Conn_01x02, J4 Qwiic_Vertical, J5 Conn_01x02, J6 Conn_01x02, J7 Conn_01x03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

Commit message: Feature/merge develop to main (#3)
* remove fix soldered tempertaure sesor

* Feature/description on soldermask (#2)

* fix Readme

* enhance README with KiBOT usage instructions and asset generation workflow

* make shure everithing is english

* improve readme

* fix upload path

* fix tittle in readme

* add silk screen and mmWave connector

* Update artifact name in fabrication workflow

* try other pr pipeline

* add more JST connectors for UART

* add jst connector for aditional gpios
Parts:
- removed C6: 100n, Capacitor_SMD:C_0805_2012Metric
- removed U3: SHT40, PCM_SparkFun-Sensor:Sensirion_DFN-4_1.5x1.5mm_P0.8mm_SHT4x_NoCentralPad
- added J13: SCD40 Module, PCM_SparkFun-Connector:1x04_P2.54mm, F.Cu at (155.2, 92.3)
- added J14: BME280, SHT40 Module, PCM_SparkFun-Connector:1x04_P2.54mm, F.Cu at (158.0, 92.3)
- added J15: mmWave Connector, PCM_SparkFun-Connector:JST_1x04_P1.0mm_Vertical_SMD, B.Cu at (96.2, 86.2)
- added J16: mmWave Connector, PCM_SparkFun-Connector:JST_1x04_P1.0mm_Vertical_SMD, F.Cu at (107.0, 74.0)
- added J17: mmWave Connector, PCM_SparkFun-Connector:JST_1x04_P1.0mm_Vertical_SMD, B.Cu at (110.5, 91.0)
- added R13: 2k2, Resistor_SMD:R_0805_2012Metric, F.Cu at (99.8, 105.5)
- added R14: 2k2, Resistor_SMD:R_0805_2012Metric, F.Cu at (122.8, 101.2)
- added R15: 2k2, Resistor_SMD:R_0805_2012Metric, F.Cu at (99.8, 101.8)
- moved R4 39.0 mm to (146.5, 84.8)
- moved R3 34.4 mm to (144.0, 84.8)
- moved R5 6.51 mm to (152.1, 77.0)
- moved Q1 6.26 mm to (157.6, 77.2)
- moved R1 4.80 mm to (149.0, 98.8), turned to 180 degrees
- moved R2 4.26 mm to (142.0, 98.8), turned to 180 degrees
- moved R8 1.56 mm to (142.0, 101.5)
- moved R7 1.00 mm to (149.0, 101.5)
- moved U2 0.50 mm to (100.5, 72.2)
Connections:
- net Net-(J12-Pin_2) renamed GPIO_6_
- net Net-(J7-Pin_2) renamed GPIO_4_
- net Net-(J8-Pin_2) renamed GPIO_5_
Routing:
- net GPIO_5_: track 3.26 -> 30.9 mm, vias 0 -> 1
- net GPIO_4_: track 6.53 -> 30.6 mm
- net UART_TX_mmWAVE: track 14.8 -> 35.5 mm
- net UART_RX_mmWAVE: track 12.5 -> 31.2 mm
- net +5V: track 76.5 -> 92.5 mm
- net GPIO_6_: track 15.1 -> 29.3 mm
- net SCK: track 122.4 -> 115.5 mm
- net Net-(J5-Pin_2): track 5.64 -> 9.66 mm
- net PIR: track 38.0 -> 41.9 mm
- net Relais: track 41.8 -> 45.2 mm
- net +3V3: track 24.4 -> 27.7 mm, vias 6 -> 7
- net SDA: track 125.1 -> 122.4 mm
- net GND: track 10.6 -> 12.3 mm
- net PhotoMeas: track 64.6 -> 63.3 mm
- net Net-(J6-Pin_2): track 6.42 -> 7.70 mm
Other:
- outline, holes or cut-outs redrawn
- board text added: "3V3"
- board text added: "3V3 |"
- board text added: "5V"
- board text added: "G1"
- board text added: "G2"
- board text added: "GND"
- board text added: "GND |"
- board text added: "GPIO 4 / 5"
- board text added: "I2C"
- board text added: "Relais"
- board text added: "SCK"
- board text added: "SDA"
- board text added: "UART"
